Commit message: fix some issues with urdf

File: urdf/barista_robot_model.urdf (robot description, URDF)
Before this commit: robot barista_robot, 16 links, 15 joints
Links:
- added link laser_scanner_frame
- link laser_scanner: geometry collision box size=0.05 0.05 0.07; visual mesh filename=package://barista_robot_description/meshes/hokuyo_urg_04lx.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 scale=1.0 1.0 1.0
Joints:
- removed joint base_joint
- added joint joint_base_link: type fixed, parent base_footprint, child base_link, origin xyz=0 0 0.0775 rpy=0 0 0
- added joint laser_scanner_frame_joint: type fixed, parent laser_scanner, child laser_scanner_frame, origin xyz=0 0 0.06 rpy=0 0 0
- joint back_left_rod_joint: origin xyz=-0.12 0.12 0.155 rpy=0 0 0 -> xyz=-0.08 0.08 0.0775 rpy=0 0 0
- joint back_right_rod_joint: origin xyz=-0.12 -0.12 0.155 rpy=0 0 0 -> xyz=-0.08 -0.08 0.0775 rpy=0 0 0
- joint back_yaw_joint: origin xyz=-0.14 0.0 -0.065 rpy=0 0 0 -> xyz=-0.14 0.0 -0.0673 rpy=0 0 0
- joint front_left_rod_joint: origin xyz=0.12 0.12 0.155 rpy=0 0 0 -> xyz=0.08 0.08 0.0775 rpy=0 0 0
- joint front_right_rod_joint: origin xyz=0.12 -0.12 0.155 rpy=0 0 0 -> xyz=0.08 -0.08 0.0775 rpy=0 0 0
- joint front_yaw_joint: origin xyz=0.14 0.0 -0.065 rpy=0 0 0 -> xyz=0.14 0.0 -0.0673 rpy=0 0 0
- joint laser_scanner_joint: origin xyz=0.03 0.0 0.205 rpy=0 0 0 -> xyz=0.03 0.0 0.0775 rpy=0 0 0
- joint left_wheel_joint: origin xyz=0.0 0.15 0.0 rpy=-1.5708 0 0 -> xyz=0 0.15 -0.0423 rpy=0 0 0
- joint right_wheel_joint: origin xyz=0.0 -0.15 0.0 rpy=-1.5708 0 0 -> xyz=0 -0.15 -0.0423 rpy=0 0 0
- joint tray_joint: origin xyz=0 0 0.375 rpy=0 0 0 -> xyz=0 0 0.2975 rpy=0 0 0

Commit message: Scanner just front

File: urdf/barista_robot_model.urdf (robot description, URDF)
Before this commit: robot barista_robot, 17 links, 16 joints
Joints:
- removed joint joint_base_link
- added joint base_link_joint: type fixed, parent base_footprint, child base_link, origin xyz=0 0 0.0775 rpy=0 0 0
- joint laser_scanner_joint: origin xyz=0.03 0.0 0.0775 rpy=0 0 0 -> xyz=0.12 0.0 0.0775 rpy=0 0 0
- joint left_wheel_joint: origin xyz=0 0.15 -0.0423 rpy=0 0 0 -> xyz=0 0.15 -0.0623 rpy=0 0 0
- joint right_wheel_joint: origin xyz=0 -0.15 -0.0423 rpy=0 0 0 -> xyz=0 -0.15 -0.0623 rpy=0 0 0
