Commit message: add namespace with robot name for xacro

File: xacro/barista_robot_model.urdf.xacro (robot description, xacro)
@@ -3,4 +3,6 @@
   <!-- Argument for conditionally including laser scanner -->
   <xacro:arg name="include_laser" default="true"/>
+  <!-- Argument for robot name -->
+  <xacro:property name="robot_name" value="$(arg robot_name)"/>
   <!-- Include all macro files -->
   <xacro:include filename="$(find barista_robot_description)/xacro/drive_wheel.xacro"/>
@@ -25,4 +27,13 @@
     <color rgba="0 1 0 1"/>
   </material>
+  <!-- Conditional color based on robot name -->
+  <xacro:if value="${robot_name == 'rick'}">
+    <xacro:property name="robot_color" value="red"/>
+    <xacro:property name="gazebo_color" value="Gazebo/Red"/>
+  </xacro:if>
+  <xacro:unless value="${robot_name == 'rick'}">
+    <xacro:property name="robot_color" value="blue"/>
+    <xacro:property name="gazebo_color" value="Gazebo/Blue"/>
+  </xacro:unless>
   <!-- Base Footprint Link -->
   <link name="base_footprint"/>
@@ -33,5 +44,5 @@
         <cylinder radius="0.178" length="0.155"/>
       </geometry>
-      <material name="blue"/>
+      <material name="${robot_color}"/>
     </visual>
     <collision>
@@ -54,5 +65,5 @@
   <!-- Gazebo Properties for Base Link -->
   <gazebo reference="base_link">
-    <material>Gazebo/Blue</material>
+    <material>${gazebo_color}</material>
   </gazebo>
   <!-- Drive Wheels -->
@@ -89,5 +100,5 @@
   <!-- Laser Scanner (conditional) -->
   <xacro:if value="$(arg include_laser)">
-    <xacro:laser_scanner parent_link="base_link">
+    <xacro:laser_scanner parent_link="base_link" robot_name="${robot_name}">
       <origin xyz="0.12 0.0 0.0775" rpy="0 0 0"/>
     </xacro:laser_scanner>
@@ -98,4 +109,5 @@
     <plugin name="barista_bot_joint_state" filename="libgazebo_ros_joint_state_publisher.so">
       <ros>
+        <namespace>/${robot_name}</namespace>
         <remapping>~/out:=joint_states</remapping>
       </ros>
@@ -114,4 +126,8 @@
   <gazebo>
     <plugin name="differential_drive_controller" filename="libgazebo_ros_diff_drive.so">
+      <ros>
+        <namespace>/${robot_name}</namespace>
+        <remapping>/cmd_vel:=cmd_vel</remapping>
+      </ros>
       <!-- wheels -->
       <left_joint>left_wheel_joint</left_joint>
@@ -126,6 +142,6 @@
       <publish_odom>true</publish_odom>
       <publish_odom_tf>true</publish_odom_tf>
-      <odometry_frame>odom</odometry_frame>
-      <robot_base_frame>base_footprint</robot_base_frame>
+      <odometry_frame>${robot_name}/odom</odometry_frame>
+      <robot_base_frame>${robot_name}/base_footprint</robot_base_frame>
       <update_rate>30</update_rate>
     </plugin>

File: xacro/laser_scanner.xacro (robot description, xacro)
@@ -7,5 +7,5 @@
   <xacro:property name="laser_box_z" value="0.07"/>
   <!-- Laser Scanner Macro -->
-  <xacro:macro name="laser_scanner" params="parent_link *origin">
+  <xacro:macro name="laser_scanner" params="parent_link robot_name *origin">
     <!-- Laser Scanner Link -->
     <link name="laser_scanner">
@@ -77,8 +77,9 @@
         <plugin name="laser" filename="libgazebo_ros_ray_sensor.so">
           <ros>
+            <namespace>/${robot_name}</namespace>
             <remapping>~/out:=scan</remapping>
           </ros>
           <output_type>sensor_msgs/LaserScan</output_type>
-          <frame_name>laser_scanner_frame</frame_name>
+          <frame_name>${robot_name}/laser_scanner_frame</frame_name>
         </plugin>
       </sensor>

Commit message: Use diff colors for laser in gazebo

File: xacro/barista_robot_model.urdf.xacro (robot description, xacro)
@@ -31,8 +31,10 @@
     <xacro:property name="robot_color" value="red"/>
     <xacro:property name="gazebo_color" value="Gazebo/Red"/>
+    <xacro:property name="laser_color" value="Gazebo/Red"/>
   </xacro:if>
   <xacro:unless value="${robot_name == 'rick'}">
     <xacro:property name="robot_color" value="blue"/>
     <xacro:property name="gazebo_color" value="Gazebo/Blue"/>
+    <xacro:property name="laser_color" value="Gazebo/Blue"/>
   </xacro:unless>
   <!-- Base Footprint Link -->
@@ -100,5 +102,5 @@
   <!-- Laser Scanner (conditional) -->
   <xacro:if value="$(arg include_laser)">
-    <xacro:laser_scanner parent_link="base_link" robot_name="${robot_name}">
+    <xacro:laser_scanner parent_link="base_link" robot_name="${robot_name}" laser_color="${laser_color}">
       <origin xyz="0.12 0.0 0.0775" rpy="0 0 0"/>
     </xacro:laser_scanner>

File: xacro/laser_scanner.xacro (robot description, xacro)
@@ -7,5 +7,5 @@
   <xacro:property name="laser_box_z" value="0.07"/>
   <!-- Laser Scanner Macro -->
-  <xacro:macro name="laser_scanner" params="parent_link robot_name *origin">
+  <xacro:macro name="laser_scanner" params="parent_link robot_name laser_color *origin">
     <!-- Laser Scanner Link -->
     <link name="laser_scanner">
@@ -26,11 +26,5 @@
         <mass value="${laser_mass}"/>
         <!-- Box inertia: Ixx = (1/12)*m*(y^2 + z^2), Iyy = (1/12)*m*(x^2 + z^2), Izz = (1/12)*m*(x^2 + y^2) -->
-        <inertia
-          ixx="${(1/12) * laser_mass * (laser_box_y * laser_box_y + laser_box_z * laser_box_z)}"
-          ixy="0.0"
-          ixz="0.0"
-          iyy="${(1/12) * laser_mass * (laser_box_x * laser_box_x + laser_box_z * laser_box_z)}"
-          iyz="0.0"
-          izz="${(1/12) * laser_mass * (laser_box_x * laser_box_x + laser_box_y * laser_box_y)}"/>
+        <inertia ixx="${(1/12) * laser_mass * (laser_box_y * laser_box_y + laser_box_z * laser_box_z)}" ixy="0.0" ixz="0.0" iyy="${(1/12) * laser_mass * (laser_box_x * laser_box_x + laser_box_z * laser_box_z)}" iyz="0.0" izz="${(1/12) * laser_mass * (laser_box_x * laser_box_x + laser_box_y * laser_box_y)}"/>
       </inertial>
     </link>
@@ -75,4 +69,5 @@
         <visualize>true</visualize>
         <update_rate>100.0</update_rate>
+        <material>${laser_color}</material>
         <plugin name="laser" filename="libgazebo_ros_ray_sensor.so">
           <ros>

Commit message: Fix some issues with robots

File: xacro/barista_robot_model.urdf.xacro (robot description, xacro)
@@ -4,4 +4,5 @@
   <xacro:arg name="include_laser" default="true"/>
   <!-- Argument for robot name -->
+  <xacro:arg name="robot_name" default="rick"/>
   <xacro:property name="robot_name" value="$(arg robot_name)"/>
   <!-- Include all macro files -->
@@ -97,5 +98,5 @@
   </xacro:standoff_rod>
   <!-- Cup Holder Tray -->
-  <xacro:cup_holder_tray parent_link="base_link">
+  <xacro:cup_holder_tray parent_link="base_link" robot_color="${robot_color}" gazebo_color="${gazebo_color}">
     <origin xyz="0 0 0.2975" rpy="0 0 0"/>
   </xacro:cup_holder_tray>

File: xacro/cup_holder_tray.xacro (robot description, xacro)
@@ -6,5 +6,5 @@
   <xacro:property name="tray_mass" value="2.0"/>
   <!-- Cup Holder Tray Macro -->
-  <xacro:macro name="cup_holder_tray" params="parent_link *origin">
+  <xacro:macro name="cup_holder_tray" params="parent_link robot_color gazebo_color *origin">
     <!-- Cup Holder Tray Link -->
     <link name="cup_holder_tray">
@@ -14,5 +14,5 @@
           <cylinder radius="${tray_radius}" length="${tray_height}"/>
         </geometry>
-        <material name="blue"/>
+        <material name="${robot_color}"/>
       </visual>
       <collision>
@@ -26,11 +26,5 @@
         <mass value="${tray_mass}"/>
         <!-- Cylinder inertia: Ixx = Iyy = (1/12)*m*(3*r^2 + h^2), Izz = (1/2)*m*r^2 -->
-        <inertia
-          ixx="${(1/12) * tray_mass * (3 * tray_radius * tray_radius + tray_height * tray_height)}"
-          ixy="0.0"
-          ixz="0.0"
-          iyy="${(1/12) * tray_mass * (3 * tray_radius * tray_radius + tray_height * tray_height)}"
-          iyz="0.0"
-          izz="${(1/2) * tray_mass * tray_radius * tray_radius}"/>
+        <inertia ixx="${(1/12) * tray_mass * (3 * tray_radius * tray_radius + tray_height * tray_height)}" ixy="0.0" ixz="0.0" iyy="${(1/12) * tray_mass * (3 * tray_radius * tray_radius + tray_height * tray_height)}" iyz="0.0" izz="${(1/2) * tray_mass * tray_radius * tray_radius}"/>
       </inertial>
     </link>
@@ -43,5 +37,5 @@
     <!-- Gazebo Properties -->
     <gazebo reference="cup_holder_tray">
-      <material>Gazebo/Blue</material>
+      <material>${gazebo_color}</material>
     </gazebo>
   </xacro:macro>
